File: PicoBPSK.kicad_sch (KiCad schematic)
At the start: 27 parts, among them SW2 RUN, SW3 BOOTSEL, SW4 IO3, U5 RP2354A

Commit message: add debug if
Parts:
- added J7: Conn_01x03, Connector_PinHeader_2.54mm:PinHeader_1x03_P2.54mm_Vertical, symbol Connector_Generic:Conn_01x03
Connections:
- net GND: now also J7.2 (Pin_2)
- new net SWCLK: J7.1 (Pin_1)
- new net SWDIO: J7.3 (Pin_3)
Other:
- note added: "Debug I/F"
