File: PicoBPSK.kicad_sch (KiCad schematic)
At the start: 28 parts, among them J7 Conn_01x03, SW2 RUN, SW3 BOOTSEL, SW4 IO3, U5 RP2354A

Commit message: add xtal
Parts:
- added C4, C5: 15p, Capacitor_SMD:C_0603_1608Metric, symbol Device:C
- added R21: 0, Resistor_SMD:R_0603_1608Metric, symbol Device:R
- added R5: 1k, Resistor_SMD:R_0603_1608Metric, symbol Device:R
- added Y1: 12MHz, Crystal:Crystal_SMD_3225-4Pin_3.2x2.5mm, symbol Device:Crystal_GND24
Connections:
- net GND: now also C4.2, C5.2, Y1.2 (G), Y1.4 (G)
- net SWCLK: now also U5.24 (SWCLK)
- net SWDIO: now also U5.25 (SWDIO)
- net XIN: now reaches U5.21 (XIN)
- net XIN: now also R21.2
- net XOUT: now reaches U5.22 (XOUT)
- net XOUT: now also R5.2
- new net: C4.1, R21.1, Y1.1
- new net: C5.1, R5.1, Y1.3
Other:
- note added: "Clock"
- moved on the sheet: R8, R9

Commit message: fix error
Parts:
- added C6: 4.7u, Capacitor_SMD:C_0603_1608Metric, symbol Device:C
- added R22: 200, Resistor_SMD:R_0603_1608Metric, symbol Device:R
- added R23: 1, Resistor_SMD:R_0603_1608Metric, symbol Device:R
Connections:
- net RUN is gone; now on net ~{RUN}: R4.2
- net +3V3: now also R22.2
- net GND: now also C6.2
- net ~{QSPI_SS}: now also U5.60 (~{QSPI_SS})
- net AVDD: now reaches U5.44 (ADC_AVDD)
- net AVDD: now also C6.1, R23.1
- new net VREF: R22.1, R23.2
- no-connect marks 3 -> 39
Other:
- note added: "USB Power"

Commit message: fix error of power line
Other:
- note added: "for DVDD"
- note added: "for IOVDD"
Changed lines of the file:
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@@
 		(comment 1 "USB-BPSK Converter Using RP2354")
+	)
+	(text "for IOVDD"
+		(exclude_from_sim no)
+		(at 95.25 39.624 0)
+		(effects
+			(font
+				(size 1.27 1.27)
+			)
+		)
+	)
+	(text "for DVDD"
+		(exclude_from_sim no)
+		(at 107.95 65.024 0)
+		(effects
+			(font
+				(size 1.27 1.27)
+			)
+		)
 	)
 	(text "Input - Switch"
@@
 		)
 	)
+	(text "for IOVDD"
+		(exclude_from_sim no)
+		(at 69.85 65.024 0)
+		(effects
+			(font
+				(size 1.27 1.27)
+			)
+		)
+	)

Commit message: add bpsk sheet
Other:
- added sheet bpsk (bpsk.kicad_sch)
- note added: "BPSK"
Changed lines of the file:
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@@
 		)
 	)
+	(text "BPSK"
+		(exclude_from_sim no)
+		(at 247.65 88.9 0)
+		(effects
+			(font
+				(size 3.81 3.81)
+			)
+		)
+	)
 	(text "Input - Switch"
 		(exclude_from_sim no)
@@
 				)
 			)
+		)
+	)
+	(sheet
+		(at 228.6 76.2)
+		(size 38.1 25.4)
+		(exclude_from_sim no)
+		(in_bom yes)
+		(on_board yes)
+		(dnp no)
+		(fields_autoplaced yes)
+		(stroke
+			(width 0.1524)
+			(type solid)
+		)
+		(fill
+			(color 0 0 0 0)
+		)
+		(property "Sheetname" "bpsk"
+			(at 228.6 75.4884 0)
+			(show_name no)
+			(do_not_autoplace no)
+			(effects
+				(font
+					(size 1.27 1.27)
+				)
+				(justify left bottom)
+			)
+		)
+		(property "Sheetfile" "bpsk.kicad_sch"
+			(at 228.6 102.1846 0)
+			(show_name no)
+			(do_not_autoplace no)
+			(effects
+				(font
+					(size 1.27 1.27)
+				)
+				(justify left top)
+			)
+		)
+		(instances
+			(project "PicoBPSK"
+				(path "/2bd032f8-7511-456b-b52b-94ead8598334"
+					(page "3")
+				)
+			)

Commit message: update bpsk sch
Other:
- sheet bpsk ports: added RX_LEV_H, RX_LEV_L, RX_SIG, RX_SIG_H, RX_SIG_L, TX_FET_D, TX_FET_U, TX_LEV_H, TX_LEV_L; removed none
Changed lines of the file:
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@@
+			)
+		)
+		(pin "RX_LEV_H" input
+			(at 228.6 88.9 180)
+			(effects
+				(font
+					(size 1.27 1.27)
+				)
+				(justify left)
+			)
+		)
+		(pin "RX_LEV_L" input
+			(at 228.6 91.44 180)
+			(effects
+				(font
+					(size 1.27 1.27)
+				)
+				(justify left)
+			)
+		)
+		(pin "RX_SIG_H" output
+			(at 228.6 96.52 180)
+			(effects
+				(font
+					(size 1.27 1.27)
+				)
+				(justify left)
+			)
+		)
+		(pin "RX_SIG_L" output
+			(at 228.6 99.06 180)
+			(effects
+				(font
+					(size 1.27 1.27)
+				)
+				(justify left)
+			)
+		)
+		(pin "TX_FET_D" input
+			(at 228.6 81.28 180)
+			(effects
+				(font
+					(size 1.27 1.27)
+				)
+				(justify left)
+			)
+		)
+		(pin "TX_FET_U" input
+			(at 228.6 78.74 180)
+			(effects
+				(font
+					(size 1.27 1.27)
+				)
+				(justify left)
+			)
+		)
+		(pin "TX_LEV_H" input
+			(at 228.6 83.82 180)
+			(effects
+				(font
+					(size 1.27 1.27)
+				)
+				(justify left)
+			)
+		)
+		(pin "TX_LEV_L" input
+			(at 228.6 86.36 180)
+			(effects
+				(font
+					(size 1.27 1.27)
+				)
+				(justify left)
+			)
+		)
+		(pin "RX_SIG" output
+			(at 228.6 93.98 180)
+			(effects
+				(font
+					(size 1.27 1.27)
+				)
+				(justify left)
 			)
 		)

Commit message: add signals
Other:
- sheet bpsk ports: added RX_ADC_SIG, RX_CMP_H, RX_CMP_L; removed RX_SIG, RX_SIG_H, RX_SIG_L
Changed lines of the file:
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@@
 			)
 		)
-		(pin "RX_SIG_H" output
-			(at 228.6 96.52 180)
+		(pin "RX_CMP_H" output
+			(at 266.7 93.98 0)
 			(effects
 				(font
 					(size 1.27 1.27)
 				)
-				(justify left)
+				(justify right)
 			)
 		)
-		(pin "RX_SIG_L" output
-			(at 228.6 99.06 180)
+		(pin "RX_CMP_L" output
+			(at 266.7 96.52 0)
 			(effects
 				(font
 					(size 1.27 1.27)
 				)
-				(justify left)
+				(justify right)
 			)
 		)
@@
 			)
 		)
-		(pin "RX_SIG" output
-			(at 228.6 93.98 180)
+		(pin "RX_ADC_SIG" output
+			(at 266.7 91.44 0)
 			(effects
 				(font
 					(size 1.27 1.27)
 				)
-				(justify left)
+				(justify right)
 			)
 		)

Commit message: update tx sch
Other:
- sheet bpsk ports: added RX_LEV_[0..3]; removed RX_LEV_H, RX_LEV_L
Changed lines of the file:
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@@
-			)
-		)
-		(pin "RX_LEV_H" input
-			(at 228.6 88.9 180)
-			(effects
-				(font
-					(size 1.27 1.27)
-				)
-				(justify left)
-			)
-		)
-		(pin "RX_LEV_L" input
-			(at 228.6 91.44 180)
-			(effects
-				(font
-					(size 1.27 1.27)
-				)
-				(justify left)
 			)
 		)
@@
 			)
 		)
+		(pin "RX_LEV_[0..3]" input
+			(at 228.6 93.98 180)
+			(effects
+				(font
+					(size 1.27 1.27)
+				)
+				(justify left)
+			)
+		)

Commit message: update comment
Other:
- sheet bpsk ports: added TX_FET_N, TX_FET_P, TX_LEV_[0..1]; removed TX_FET_D, TX_FET_U, TX_LEV_H, TX_LEV_L
Changed lines of the file:
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@@
 	(wire
 		(pts
+			(xy 152.4 39.37) (xy 149.86 39.37)
+		)
+		(stroke
+			(width 0)
+			(type default)
+		)
+	)
+	(wire
+		(pts
 			(xy 76.2 25.4) (xy 82.55 25.4)
 		)
@@
 	(wire
 		(pts
-			(xy 149.86 38.1) (xy 149.86 43.18)
+			(xy 152.4 38.1) (xy 152.4 39.37)
 		)
 		(stroke
@@
 	(wire
 		(pts
+			(xy 266.7 93.98) (xy 276.86 93.98)
+		)
+		(stroke
+			(width 0)
+			(type default)
+		)
+	)
+	(wire
+		(pts
 			(xy 101.6 111.76) (xy 101.6 114.3)
 		)
@@
 	(wire
 		(pts
+			(xy 266.7 96.52) (xy 276.86 96.52)
+		)
+		(stroke
+			(width 0)
+			(type default)
+		)
+	)
+	(wire
+		(pts
 			(xy 187.96 63.5) (xy 177.8 63.5)
 		)
@@
 		)
 	)
+	(bus
+		(pts
+			(xy 218.44 78.74) (xy 228.6 78.74)
+		)
+		(stroke
+			(width 0)
+			(type default)
+		)
+	)
+	(wire
+		(pts
+			(xy 149.86 39.37) (xy 149.86 43.18)
+		)
+		(stroke
+			(width 0)
+			(type default)
+		)
+	)
 	(wire
 		(pts
@@
 	(wire
 		(pts
+			(xy 218.44 85.09) (xy 228.6 85.09)
+		)
+		(stroke
+			(width 0)
+			(type default)
+		)
+	)
+	(wire
+		(pts
+			(xy 218.44 82.55) (xy 228.6 82.55)
+		)
+		(stroke
+			(width 0)
+			(type default)
+		)
+	)
+	(wire
+		(pts
 			(xy 60.96 165.1) (xy 71.12 165.1)
 		)
@@
 	(wire
 		(pts
+			(xy 266.7 91.44) (xy 276.86 91.44)
+		)
+		(stroke
+			(width 0)
+			(type default)
+		)
+	)
+	(wire
+		(pts
 			(xy 187.96 66.04) (xy 177.8 66.04)
 		)
@@
 		)
 	)
+	(bus
+		(pts
+			(xy 218.44 93.98) (xy 228.6 93.98)
+		)
+		(stroke
+			(width 0)
+			(type default)
+		)
+	)
 	(label "~{RUN}"
 		(at 71.12 165.1 180)
@@
 	(symbol
 		(lib_id "power:+3V3")
-		(at 149.86 38.1 0)
+		(at 152.4 38.1 0)
 		(unit 1)
 		(body_style 1)
@@
 		(fields_autoplaced yes)
 		(property "Reference" "#PWR024"
-			(at 149.86 41.91 0)
+			(at 152.4 41.91 0)
 			(hide yes)
 			(show_name no)
@@
 		)
 		(property "Value" "+3V3"
-			(at 149.86 33.02 0)
+			(at 152.4 33.02 0)
 			(show_name no)
 			(do_not_autoplace no)
@@
 		)
 		(property "Footprint" ""
-			(at 149.86 38.1 0)
+			(at 152.4 38.1 0)
 			(hide yes)
 			(show_name no)
@@
 		)
 		(property "Datasheet" ""
-			(at 149.86 38.1 0)
+			(at 152.4 38.1 0)
 			(hide yes)
 			(show_name no)
@@
 		)
 		(property "Description" "Power symbol creates a global label with name \"+3V3\""
-			(at 149.86 38.1 0)
+			(at 152.4 38.1 0)
 			(hide yes)
 			(show_name no)
@@
 			)
 		)
-		(pin "TX_FET_D" input
-			(at 228.6 81.28 180)
+		(pin "TX_FET_N" input
+			(at 228.6 85.09 180)
 			(effects
 				(font
@@
 			)
 		)
-		(pin "TX_FET_U" input
-			(at 228.6 78.74 180)
+		(pin "TX_FET_P" input
+			(at 228.6 82.55 180)
 			(effects
 				(font
@@
 			)
 		)
-		(pin "TX_LEV_H" input
-			(at 228.6 83.82 180)
+		(pin "RX_ADC_SIG" output
+			(at 266.7 91.44 0)
 			(effects
 				(font
 					(size 1.27 1.27)
 				)
-				(justify left)
+				(justify right)
 			)
 		)
-		(pin "TX_LEV_L" input
-			(at 228.6 86.36 180)
+		(pin "RX_LEV_[0..3]" input
+			(at 228.6 93.98 180)
 			(effects
 				(font
@@
 			)
 		)
-		(pin "RX_ADC_SIG" output
-			(at 266.7 91.44 0)
-			(effects
-				(font
-					(size 1.27 1.27)
-				)
-				(justify right)
-			)
-		)
-		(pin "RX_LEV_[0..3]" input
-			(at 228.6 93.98 180)
+		(pin "TX_LEV_[0..1]" input
+			(at 228.6 78.74 180)
 			(effects
 				(font
