File: PicoBPSK.kicad_sch (KiCad schematic)
At the start: 36 parts, among them J7 Conn_01x03, SW2 RUN, SW3 BOOTSEL, SW4 IO3, U5 RP2354A, Y1 12MHz

Commit message: add TP
Parts:
- added LD5: ERR, LED_SMD:LED_0603_1608Metric, symbol Device:LED
- added LD6: RX, LED_SMD:LED_0603_1608Metric, symbol Device:LED
- added LD7: TX, LED_SMD:LED_0603_1608Metric, symbol Device:LED
- added Q13, Q14, Q15: AO3400A, Package_TO_SOT_SMD:SOT-23, symbol Transistor_FET:AO3400A
- added R41, R62, R64: 1k, Resistor_SMD:R_0603_1608Metric, symbol Device:R
- added R63, R65, R66: 10k, Resistor_SMD:R_0603_1608Metric, symbol Device:R
- J7: value Conn_01x03 -> SWD
Connections:
- net IO3 is gone; now on net SW: C9.2, R7.2, SW4.2
- net +3V3: now also R41.2, R62.2, R63.2, R64.2
- net GND: now also Q13.2 (S), Q14.2 (S), Q15.2 (S), R65.1, R66.1
- net TX_LEV_0: now reaches U5.14 (GPIO10)
- net TX_LEV_1: now reaches U5.15 (GPIO11)
- net TX_FET_P: now reaches U5.16 (GPIO12)
- net TX_FET_N: now reaches U5.17 (GPIO13)
- net SW: now reaches U5.2 (GPIO0)
- net Err: now reaches U5.3 (GPIO1)
- net Err: now also Q13.1 (G), R63.1
- net RX_LEV_0: now reaches U5.32 (GPIO20)
- net RX_LEV_1: now reaches U5.33 (GPIO21)
- net RX_LEV_2: now reaches U5.34 (GPIO22)
- net RX_LEV_3: now reaches U5.35 (GPIO23)
- net RX_CMP_H: now reaches U5.36 (GPIO24)
- net RX_CMP_L: now reaches U5.37 (GPIO25)
- net RX: now reaches U5.4 (GPIO2)
- net RX: now also Q14.1 (G), R65.2
- net RX_ADC_S: now reaches U5.40 (GPIO26/ADC0)
- net TX: now reaches U5.5 (GPIO3)
- net TX: now also Q15.1 (G), R66.2
- new net: LD7.2 (A), R64.1
- new net: LD6.2 (A), R62.1
- new net: LD5.2 (A), R41.1
- new net: LD7.1 (K), Q15.3 (D)
- new net: LD5.1 (K), Q13.3 (D)
- new net: LD6.1 (K), Q14.3 (D)
- no-connect marks 39 -> 24
Other:
- sheet bpsk ports: added RX_ADC_S; removed RX_ADC_SIG
- note added: "Blue"
- note added: "Color LCSC# name isBaic wavelength Red C2286 KT-0603R o 620 Yellow C2289 xxxx o 589 White C2290 KT-0603W o --- Green C12624 KT-0603G x 525 Blue C2288 KT-0603B x 469 YGreen C2289 KT-0603YG x 576"
- note added: "Output - LED"
- note added: "Power"
- note added: "Red"
- moved on the sheet: H1, H2, H3, H4, J7

Commit message: update fotprint
Parts:
- LD5: LCSC C12624 -> C2286
- LD6, LD7: LCSC C12624 -> C2289
Other:
- note added: "Yellow"
- note removed: "Blue"
Changed lines of the file:
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@@
 		)
 	)
-	(text "Blue"
+	(text "Yellow"
 		(exclude_from_sim no)
 		(at 270.51 124.968 0)
@@
 		)
 	)
-	(text "Blue"
+	(text "Yellow"
 		(exclude_from_sim no)
 		(at 245.11 124.968 0)
@@
 			)
 		)
-		(property "LCSC" "C12624"
+		(property "LCSC" "C2289"
 			(at 266.7 120.65 90)
 			(hide yes)
@@
 			)
 		)
-		(property "LCSC" "C12624"
+		(property "LCSC" "C2289"
 			(at 241.3 120.65 90)
 			(hide yes)
@@
 			)
 		)
-		(property "LCSC" "C12624"
+		(property "LCSC" "C2286"
 			(at 215.9 120.65 90)
 			(hide yes)

Commit message: update part num
Parts:
- removed R23: 1, Resistor_SMD:R_0603_1608Metric, symbol Device:R
- added C17: 100n, Capacitor_SMD:C_0402_1005Metric, symbol Device:C
- C15: renamed from C6; value 4.7u -> 2.2u
- R6: renamed from R22; value 200 -> 22
- SW3: renamed from SW4; value IO3 -> SW
- renumbered C4 to C1, C27 to C10, C24 to C11, C16 to C12, C15 to C13, C7 to C14, C17 to C16, C9 to C18, C28 to C2, C20 to C3, C25 to C4, C3 to C6, C21 to C7, C26 to C8, C23 to C9, J7 to J1, LD5 to LD1, LD6 to LD2, LD7 to LD3, Q13 to Q1, Q14 to Q2, Q15 to Q3, R4 to R1, R41 to R10, R65 to R11, R62 to R12, R66 to R13, R64 to R14, R21 to R2, R5 to R3, R9 to R4, R8 to R5, R6 to R7, R7 to R8, R63 to R9, SW2 to SW1, SW3 to SW2, U5 to U1
Connections:
- net VREF is gone; now on an unnamed net: R6.1
- net GND: now also C17.2
- net AVDD: no longer names the net of C15.1, U1.44 (ADC_AVDD)
- net AVDD: now also C17.1
Other:
- moved on the sheet: C11, C15, C3, C7, C9, R6

Commit message: add v0.02
Parts:
- C15: LCSC (none) -> C23630; akizuki (none) -> x
- Q1, Q2, Q3: LCSC (none) -> C20917; akizuki (none) -> x
- R4, R5, R6: LCSC (none) -> C23345; akizuki (none) -> x
Changed lines of the file:
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@@
 	(title_block
 		(title "PicoBPSK")
-		(date "2026-09-03")
-		(rev "0.01")
+		(date "2026-09-07")
+		(rev "0.02")
 		(company "okdwtr")
 		(comment 1 "USB-BPSK Converter Using RP2354")
@@
 			)
 		)
-		(property "LCSC" ""
+		(property "LCSC" "C23630"
 			(at 107.95 31.75 0)
 			(hide yes)
@@
 			)
 		)
-		(property "akizuki" ""
+		(property "akizuki" "x"
 			(at 107.95 31.75 0)
 			(hide yes)
@@
 			)
 		)
+		(property "LCSC" "C20917"
+			(at 264.16 133.35 0)
+			(hide yes)
+			(show_name no)
+			(do_not_autoplace no)
+			(effects
+				(font
+					(size 1.27 1.27)
+				)
+			)
+		)
+		(property "akizuki" "x"
+			(at 264.16 133.35 0)
+			(hide yes)
+			(show_name no)
+			(do_not_autoplace no)
+			(effects
+				(font
+					(size 1.27 1.27)
+				)
+			)
+		)
 		(pin "1"
 		)
@@
 			)
 		)
-		(property "LCSC" ""
+		(property "LCSC" "C23345"
 			(at 82.55 99.06 90)
 			(hide yes)
@@
 			)
 		)
-		(property "akizuki" ""
+		(property "akizuki" "x"
 			(at 82.55 99.06 90)
 			(hide yes)
@@
 			)
 		)
-		(property "LCSC" ""
+		(property "LCSC" "C23345"
 			(at 82.55 88.9 90)
 			(hide yes)
@@
 			)
 		)
-		(property "akizuki" ""
+		(property "akizuki" "x"
 			(at 82.55 88.9 90)
 			(hide yes)
@@
 			)
 		)
+		(property "LCSC" "C20917"
+			(at 213.36 133.35 0)
+			(hide yes)
+			(show_name no)
+			(do_not_autoplace no)
+			(effects
+				(font
+					(size 1.27 1.27)
+				)
+			)
+		)
+		(property "akizuki" "x"
+			(at 213.36 133.35 0)
+			(hide yes)
+			(show_name no)
+			(do_not_autoplace no)
+			(effects
+				(font
+					(size 1.27 1.27)
+				)
+			)
+		)
 		(pin "1"
 		)
@@
 			)
 		)
+		(property "LCSC" "C20917"
+			(at 238.76 133.35 0)
+			(hide yes)
+			(show_name no)
+			(do_not_autoplace no)
+			(effects
+				(font
+					(size 1.27 1.27)
+				)
+			)
+		)
+		(property "akizuki" "x"
+			(at 238.76 133.35 0)
+			(hide yes)
+			(show_name no)
+			(do_not_autoplace no)
+			(effects
+				(font
+					(size 1.27 1.27)
+				)
+			)
+		)
 		(pin "1"
 		)
@@
 			)
 		)
-		(property "LCSC" ""
+		(property "LCSC" "C23345"
 			(at 101.6 25.4 0)
 			(hide yes)
@@
 			)
 		)
-		(property "akizuki" ""
+		(property "akizuki" "x"
 			(at 101.6 25.4 90)
 			(hide yes)
