File: bpsk.kicad_sch (KiCad schematic)
At the start: 0 parts

Commit message: update bpsk sch
Parts:
- added C1, C8: 47n, symbol Device:C
- added C18: 100n, symbol Device:C
- added C2: 10n, symbol Device:C
- added J1: Screw_Terminal_01x03, symbol Connector:Screw_Terminal_01x03
- added L1: L_Coupled_1243, symbol Device:L_Coupled_1243
- added L2, L3: L_Ferrite, symbol Device:L_Ferrite
- added Q1, Q3, Q6, Q7, Q8, Q9: AO3400A, Package_TO_SOT_SMD:SOT-23, symbol Transistor_FET:AO3400A
- added Q4, Q5: AO3401A, Package_TO_SOT_SMD:SOT-23, symbol Transistor_FET:AO3401A
- added R1, R2: R, symbol Device:R
- added R24, R25, R29, R30: 100, symbol Device:R
- added R26, R3: 3.6k, symbol Device:R
- added R27, R28, R41: 1k, symbol Device:R
- added R31, R32, R36, R38, R46, R47: 47k, symbol Device:R
- added R33, R34, R35, R37, R44, R45: 47, symbol Device:R
- added R39, R48: 68, symbol Device:R
- added R40, R49: 200, symbol Device:R
- added R42, R43: 30k, symbol Device:R
- added R50, R51, R52, R53: 11k, symbol Device:R
- added U1: LM393, symbol Comparator:LM393
Connections:
- new net: Q7.3 (D), R39.1
- new net: C8.2, L1.2
- new net: L1.3, R24.1, R3.1
- new net: L1.4, R25.1, R3.2
- new net: Q9.1 (G), R45.2, R47.1
- new net: Q6.1 (G), R35.2, R36.1
- new net: Q9.3 (D), R49.1
- new net: Q8.1 (G), R44.2, R46.1
- new net: Q3.1 (G), R32.1, R33.2
- new net: Q7.1 (G), R37.2, R38.1
- new net: Q3.3 (D), R29.1
- new net: Q1.1 (G), R31.1, R34.2
- new net: Q1.3 (D), R30.1
- new net: Q4.1 (G), R27.2, R30.2
- new net: Q6.3 (D), R40.1
- new net: Q5.1 (G), R28.2, R29.2
- new net: Q8.3 (D), R48.1
- new net +5V: C18.1, Q4.3 (D), Q5.3 (D), R27.1, R28.1, R42.1, R50.1, R53.1, U1.8 (V+)
- new net FG: J1.3 (Pin_3)
- new net GND: C18.2, C2.2, L1.1, Q1.2 (S), Q3.2 (S), Q6.2 (S), Q7.2 (S), Q8.2 (S), Q9.2 (S), R31.2, R32.2, R36.2, R38.2, R43.2, R46.2, R47.2, R51.2, R52.2, U1.4 (V-)
- new net LC: L2.1, L3.2, R1.2, R2.1, R39.2, R40.2, R48.2, R49.2
- new net LD: L2.2, Q5.2 (S), R2.2
- new net LU: L3.1, Q4.2 (S), R1.1
- new net RX_LEV_H: R44.1
- new net RX_LEV_L: R45.1
- new net RX_SIG: C2.1, C8.1, R42.2, R43.1, R50.2, R51.1, R52.1, R53.2, U1.2 (-), U1.3 (+), U1.5 (+), U1.6 (-)
- new net RX_SIG_H: U1.1
- new net RX_SIG_L: U1.7
- new net S+: C1.1, J1.1 (Pin_1), R24.2, R26.2
- new net S-: C1.2, J1.2 (Pin_2), R25.2, R26.1
- new net TX_FET_D: R33.1
- new net TX_FET_U: R34.1
- new net TX_LEV_H: R37.1
- new net TX_LEV_L: R35.1
- no-connect marks 0 -> 1

Commit message: add signals
Parts:
- removed C18: 100n, symbol Device:C
- removed Q8, Q9: AO3400A, Package_TO_SOT_SMD:SOT-23, symbol Transistor_FET:AO3400A
- removed R41: 1k, symbol Device:R
- removed R44, R45: 47, symbol Device:R
- removed R46, R47: 47k, symbol Device:R
- removed R48: 68, symbol Device:R
- removed R49: 200, symbol Device:R
- removed R50, R51, R52, R53: 11k, symbol Device:R
- removed U1: LM393, symbol Comparator:LM393
Connections:
- net RX_SIG renamed RX
Other:
- added sheet rx (rx.kicad_sch)
- note added: "AFE"
- note added: "Signal - Line Interface"
- note added: "Signal - Tx Level Select"
- moved on the sheet: C1, C2, C8, J1, L1, L2, L3, R1, R2, R24, R25, R26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

Commit message: update comment
Other:
- note added: "2.5V ±2.5V Rx Signal"
- note added: "Signal - Tx Output Driver"
- moved on the sheet: Q1, Q3, Q4, Q5, Q6, R27, R28, R29, R30, R31, R32, R33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

Commit message: update tx sch
Parts:
- J1: value Screw_Terminal_01x03 -> BPSK
- R1, R2: value R -> 470
Connections:
- net TX_LEV_H renamed TX_LEV_0
- net TX_LEV_L renamed TX_LEV_1
Other:
- sheet rx ports: added RX_LEV_[0..3]; removed RX_LEV_C, RX_LEV_H, RX_LEV_L
- note added: "Vth:2.5V ±129mV"
- moved on the sheet: C1, C2, C8, J1, L1, L2, L3, Q6, Q7, R1, R2, R24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

Commit message: update comment
Connections:
- net LD renamed LN
- net LU renamed LP
- net TX_FET_D renamed TX_FET_N
- net TX_FET_U renamed TX_FET_P
Other:
- note added: "I_{TX}:25.0mA_{max}"
- note added: "I_{TX}:735mA_{max}"
- note added: "LINE"
- note added: "RX"
- note added: "TX"
- note added: "V_{BIAS}:2.5V V_{RX}:±2.5V Rx Signal"
- note removed: "2.5V ±2.5V Rx Signal"
- note removed: "Vth:2.5V ±129mV"
Changed lines of the file:
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@@
 		(comment 1 "USB-BPSK Converter Using RP2354")
 	)
-	(text "Vth:2.5V ±129mV"
+	(circle
+		(center 176.53 48.26)
+		(radius 0.0001)
+		(stroke
+			(width 0)
+			(type default)
+		)
+		(fill
+			(type none)
+		)
+	)
+	(circle
+		(center 176.53 35.56)
+		(radius 0.0001)
+		(stroke
+			(width 0)
+			(type default)
+		)
+		(fill
+			(type none)
+		)
+	)
+	(text "I_{TX}:735mA_{max}"
 		(exclude_from_sim no)
 		(at 76.2 152.4 0)
@@
 		)
 	)
-	(text "2.5V ±2.5V\nRx Signal"
+	(text "LINE"
+		(exclude_from_sim no)
+		(at 184.15 69.85 0)
+		(effects
+			(font
+				(size 1.27 1.27)
+			)
+		)
+	)
+	(text "V_{BIAS}:2.5V\nV_{RX}:±2.5V\nRx Signal"
 		(exclude_from_sim no)
 		(at 127 88.9 0)
@@
 		)
 	)
+	(text "TX"
+		(exclude_from_sim no)
+		(at 171.45 57.15 0)
+		(effects
+			(font
+				(size 1.27 1.27)
+			)
+		)
+	)
 	(text "Signal - Line Interface"
 		(exclude_from_sim no)
@@
 		)
 	)
-	(text "Vth:2.5V ±129mV"
+	(text "I_{TX}:25.0mA_{max}"
 		(exclude_from_sim no)
 		(at 152.4 152.4 0)
@@
 		)
 	)
+	(text "RX"
+		(exclude_from_sim no)
+		(at 171.45 69.85 0)
+		(effects
+			(font
+				(size 1.27 1.27)
+			)
+		)
+	)
 	(junction
 		(at 127 152.4)
@@
 	(wire
 		(pts
+			(xy 139.7 25.4) (xy 165.1 25.4)
+		)
+		(stroke
+			(width 0)
+			(type default)
+		)
+	)
+	(wire
+		(pts
 			(xy 127 165.1) (xy 127 162.56)
 		)
@@
 	(wire
 		(pts
+			(xy 146.05 38.1) (xy 165.1 38.1)
+		)
+		(stroke
+			(width 0)
+			(type default)
+		)
+	)
+	(wire
+		(pts
 			(xy 165.1 50.8) (xy 175.26 50.8)
 		)
@@
 	(wire
 		(pts
+			(xy 139.7 50.8) (xy 146.05 50.8)
+		)
+		(stroke
+			(width 0)
+			(type default)
+		)
+	)
+	(wire
+		(pts
 			(xy 139.7 157.48) (xy 139.7 165.1)
 		)
@@
 	(wire
 		(pts
-			(xy 152.4 38.1) (xy 165.1 38.1)
-		)
-		(stroke
-			(width 0)
-			(type default)
-		)
-	)
-	(wire
-		(pts
 			(xy 175.26 76.2) (xy 175.26 77.47)
 		)
@@
 		)
 	)
+	(wire
+		(pts
+			(xy 146.05 38.1) (xy 146.05 50.8)
+		)
+		(stroke
+			(width 0)
+			(type default)
+		)
+	)
 	(polyline
 		(pts
@@
 	(wire
 		(pts
+			(xy 152.4 31.75) (xy 152.4 50.8)
+		)
+		(stroke
+			(width 0)
+			(type default)
+		)
+	)
+	(wire
+		(pts
 			(xy 50.8 46.99) (xy 50.8 44.45)
 		)
@@
 	(wire
 		(pts
-			(xy 152.4 25.4) (xy 165.1 25.4)
-		)
-		(stroke
-			(width 0)
-			(type default)
-		)
-	)
-	(wire
-		(pts
 			(xy 76.2 73.66) (xy 76.2 76.2)
 		)
@@
 		(pts
 			(xy 180.34 88.9) (xy 180.34 87.63)
+		)
+		(stroke
+			(width 0)
+			(type default)
+		)
+	)
+	(wire
+		(pts
+			(xy 139.7 31.75) (xy 152.4 31.75)
 		)
 		(stroke
@@
 		)
 	)
-	(label "LD"
-		(at 101.6 88.9 180)
-		(effects
-			(font
-				(size 1.27 1.27)
-			)
-			(justify right bottom)
-		)
-	)
 	(label "LC"
-		(at 152.4 38.1 0)
+		(at 139.7 50.8 0)
 		(effects
 			(font
@@
 		)
 	)
-	(label "LD"
-		(at 152.4 50.8 0)
+	(label "LN"
+		(at 139.7 31.75 0)
 		(effects
 			(font
@@
 		)
 	)
-	(label "LU"
+	(label "LP"
 		(at 101.6 44.45 180)
 		(effects
@@
 		)
 	)
-	(label "LU"
-		(at 152.4 25.4 0)
+	(label "LP"
+		(at 139.7 25.4 0)
 		(effects
 			(font
@@
 			)
 			(justify left bottom)
+		)
+	)
+	(label "LN"
+		(at 101.6 88.9 180)
+		(effects
+			(font
+				(size 1.27 1.27)
+			)
+			(justify right bottom)
 		)
 	)
@@
 		)
 	)
-	(hierarchical_label "TX_FET_U"
+	(hierarchical_label "TX_FET_P"
 		(shape input)
 		(at 38.1 44.45 180)
@@
 		)
 	)
-	(hierarchical_label "TX_FET_D"
+	(hierarchical_label "TX_FET_N"
 		(shape input)
 		(at 38.1 88.9 180)

Commit message: add TP
Parts:
- added TP1: TX_P, TestPoint:TestPoint_Keystone_5005-5009_Compact, symbol Connector:TestPoint
- added TP2: TX_N, TestPoint:TestPoint_Keystone_5005-5009_Compact, symbol Connector:TestPoint
- added TP3: BPSK_P, TestPoint:TestPoint_Keystone_5005-5009_Compact, symbol Connector:TestPoint
- added TP4: BPSK_N, TestPoint:TestPoint_Keystone_5005-5009_Compact, symbol Connector:TestPoint
Connections:
- net S+: now also TP3.1
- net S-: now also TP4.1
- net at Q4.1 (G), R27.2, R30.2: now also TP1.1
- net at Q5.1 (G), R28.2, R29.2: now also TP2.1
- net RX renamed RX_RAW
Other:
- sheet rx ports: added RX_ADC_S, RX_RAW; removed RX, RX_ADC_SIG
- moved on the sheet: Q1, Q3, R27, R28, R29, R30, R31, R32, R33, R34

Commit message: update fotprint
Parts:
- C1, C2, C8: footprint (none) -> Capacitor_SMD:C_0603_1608Metric
- R1, R2, R24, R25, R26, R27, R28, R29, R3, R30, R31, R32, R33, R34, R35, R36, R37, R38, R39, R40, R42, R43: footprint (none) -> Resistor_SMD:R_0603_1608Metric
Changed lines of the file:
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@@
 			)
 		)
-		(property "Footprint" ""
+		(property "Footprint" "Resistor_SMD:R_0603_1608Metric"
 			(at 76.2 141.478 90)
 			(hide yes)
@@
 			)
 		)
-		(property "Footprint" ""
+		(property "Footprint" "Resistor_SMD:R_0603_1608Metric"
 			(at 230.378 82.55 90)
 			(hide yes)
@@
 			)
 		)
-		(property "Footprint" ""
+		(property "Footprint" "Resistor_SMD:R_0603_1608Metric"
 			(at 125.222 158.75 90)
 			(hide yes)
@@
 			)
 		)
-		(property "Footprint" ""
+		(property "Footprint" "Capacitor_SMD:C_0603_1608Metric"
 			(at 153.3652 86.36 0)
 			(hide yes)
@@
 			)
 		)
-		(property "Footprint" ""
+		(property "Footprint" "Resistor_SMD:R_0603_1608Metric"
 			(at 31.75 90.678 90)
 			(hide yes)
@@
 			)
 		)
-		(property "Footprint" ""
+		(property "Footprint" "Capacitor_SMD:C_0603_1608Metric"
 			(at 168.91 75.2348 0)
 			(hide yes)
@@
 			)
 		)
-		(property "Footprint" ""
+		(property "Footprint" "Resistor_SMD:R_0603_1608Metric"
 			(at 201.422 82.55 90)
 			(hide yes)
@@
 			)
 		)
-		(property "Footprint" ""
+		(property "Footprint" "Resistor_SMD:R_0603_1608Metric"
 			(at 49.022 158.75 90)
 			(hide yes)
@@
 			)
 		)
-		(property "Footprint" ""
+		(property "Footprint" "Resistor_SMD:R_0603_1608Metric"
 			(at 137.922 69.85 90)
 			(hide yes)
@@
 			)
 		)
-		(property "Footprint" ""
+		(property "Footprint" "Resistor_SMD:R_0603_1608Metric"
 			(at 57.15 33.528 90)
 			(hide yes)
@@
 			)
 		)
-		(property "Footprint" ""
+		(property "Footprint" "Resistor_SMD:R_0603_1608Metric"
 			(at 163.322 31.75 90)
 			(hide yes)
@@
 			)
 		)
-		(property "Footprint" ""
+		(property "Footprint" "Resistor_SMD:R_0603_1608Metric"
 			(at 137.922 82.55 90)
 			(hide yes)
@@
 			)
 		)
-		(property "Footprint" ""
+		(property "Footprint" "Resistor_SMD:R_0603_1608Metric"
 			(at 163.322 44.45 90)
 			(hide yes)
@@
 			)
 		)
-		(property "Footprint" ""
+		(property "Footprint" "Resistor_SMD:R_0603_1608Metric"
 			(at 120.65 154.178 90)
 			(hide yes)
@@
 			)
 		)
-		(property "Footprint" ""
+		(property "Footprint" "Capacitor_SMD:C_0603_1608Metric"
 			(at 242.2652 86.36 0)
 			(hide yes)
@@
 			)
 		)
-		(property "Footprint" ""
+		(property "Footprint" "Resistor_SMD:R_0603_1608Metric"
 			(at 61.722 25.4 90)
 			(hide yes)
@@
 			)
 		)
-		(property "Footprint" ""
+		(property "Footprint" "Resistor_SMD:R_0603_1608Metric"
 			(at 31.75 46.228 90)
 			(hide yes)
@@
 			)
 		)
-		(property "Footprint" ""
+		(property "Footprint" "Resistor_SMD:R_0603_1608Metric"
 			(at 152.4 141.478 90)
 			(hide yes)
@@
 			)
 		)
-		(property "Footprint" ""
+		(property "Footprint" "Resistor_SMD:R_0603_1608Metric"
 			(at 215.9 90.678 90)
 			(hide yes)
@@
 			)
 		)
-		(property "Footprint" ""
+		(property "Footprint" "Resistor_SMD:R_0603_1608Metric"
 			(at 36.322 95.25 90)
 			(hide yes)
@@
 			)
 		)
-		(property "Footprint" ""
+		(property "Footprint" "Resistor_SMD:R_0603_1608Metric"
 			(at 61.722 69.85 90)
 			(hide yes)
@@
 			)
 		)
-		(property "Footprint" ""
+		(property "Footprint" "Resistor_SMD:R_0603_1608Metric"
 			(at 215.9 77.978 90)
 			(hide yes)
@@
 			)
 		)
-		(property "Footprint" ""
+		(property "Footprint" "Resistor_SMD:R_0603_1608Metric"
 			(at 44.45 154.178 90)
 			(hide yes)
@@
 			)
 		)
-		(property "Footprint" ""
+		(property "Footprint" "Resistor_SMD:R_0603_1608Metric"
 			(at 36.322 50.8 90)
 			(hide yes)
@@
 			)
 		)
-		(property "Footprint" ""
+		(property "Footprint" "Resistor_SMD:R_0603_1608Metric"
 			(at 57.15 77.978 90)
 			(hide yes)

Commit message: update part num
Parts:
- TP1, TP2, TP3, TP4: LCSC (none) -> x; akizuki (none) -> 107591
- renumbered C2 to C24, C8 to C25, C1 to C26, J1 to J3, L3 to L1, L1 to L3, Q6 to Q10, Q1 to Q5, Q3 to Q6, Q4 to Q8, Q5 to Q9, R34 to R26, R33 to R27, R31 to R28, R32 to R29, R37 to R30, R38 to R31, R30 to R32, R29 to R33, R27 to R34, R28 to R35, R39 to R36, R35 to R37, R36 to R38, R42 to R39, R43 to R40, R40 to R41, R1 to R42, R2 to R43, R3 to R44, R24 to R45, R25 to R46, R26 to R47
