File: bpsk.kicad_sch (KiCad schematic)
At the start: 39 parts, among them J3 BPSK, Q10 AO3400A, Q5 AO3400A, Q6 AO3400A, Q7 AO3400A, Q8 AO3401A, Q9 AO3401A

Commit message: update partname
Parts:
- renumbered C24 to C23, C25 to C24, C26 to C25, R26 to R17, R27 to R18, R28 to R19, R29 to R20, R30 to R21, R31 to R22, R32 to R23, R33 to R24, R34 to R25, R35 to R26, R36 to R27, R37 to R28, R38 to R29, R39 to R30, R40 to R31, R41 to R32, R42 to R33, R43 to R34, R44 to R35, R45 to R36, R46 to R37, R47 to R38

Commit message: add v0.02
Parts:
- added J4: 734-166, Connector_Wago:Wago_734-166_1x06_P3.50mm_Horizontal, symbol Connector_Generic:Conn_01x06
- C23: LCSC (none) -> C57112; akizuki (none) -> x
- C24, C25: LCSC (none) -> C1622; akizuki (none) -> x
- J3: value BPSK -> BPSK XH3p; footprint (none) -> Connector_JST:JST_XH_B3B-XH-A_1x03_P2.50mm_Vertical; symbol Connector:Screw_Terminal_01x03 -> Connector_Generic:Conn_01x03; LCSC (none) -> C144394; akizuki (none) -> 112248
- Q10, Q5, Q6, Q7: LCSC (none) -> C20917; akizuki (none) -> x
- Q8, Q9: LCSC (none) -> AO3401A; akizuki (none) -> x
- R17, R18, R21, R28: LCSC (none) -> C23182; akizuki (none) -> x
- R19, R20, R22, R29: LCSC (none) -> C25819; akizuki (none) -> x
- R23, R24, R36, R37: LCSC (none) -> C22775; akizuki (none) -> x
- R25, R26: LCSC (none) -> C21190; akizuki (none) -> x
- R27: LCSC (none) -> C27592; akizuki (none) -> x
- R30, R31: LCSC (none) -> C22984; akizuki (none) -> x
- R32: LCSC (none) -> C8218; akizuki (none) -> x
- R33, R34: LCSC (none) -> C23179; akizuki (none) -> x
- R35, R38: LCSC (none) -> C22980; akizuki (none) -> x
Connections:
- net FG: now also J3.2 (Pin_2), J4.3 (Pin_3); no longer J3.3 (Pin_3)
- net S+: now also J4.1 (Pin_1)
- net S-: now also J3.3 (Pin_3), J4.2 (Pin_2); no longer J3.2 (Pin_2)
- no-connect marks 1 -> 4
