File: usb.kicad_sch (KiCad schematic)
At the start: 33 parts, among them J2 USB FS, Q2 BSS138, U10 AMS1117-3.3, U4 TLV70012_SOT23-5, U6 CH221K, U7 CH224K, U8 R-78E3.3-1.0, U9 MAX809S

Commit message: add TP
Parts:
- removed Q2: BSS138, Package_TO_SOT_SMD:SOT-23, symbol Transistor_FET:BSS138
- added Q12: AO3400A, Package_TO_SOT_SMD:SOT-23, symbol Transistor_FET:AO3400A
- C10, LD3, R11, R12, R13, R14, R15, U7: now not fitted; now left out of the parts list
- JP2, JP3, JP4: now not fitted
Connections:
- net GND: now also Q12.2 (S)
- net RUN: now also Q12.3 (D)
- net at U9.2 (~{RESET}): now also Q12.1 (G)
- net VBUS renamed +5V

Commit message: update part num
Parts:
- renumbered C10 to C19, C11 to C20, C13 to C21, C12 to C22, C14 to C23, JP2 to JP1, JP3 to JP2, JP4 to JP3, JP5 to JP4, JP6 to JP5, JP7 to JP6, JP10 to JP7, LD3 to LD4, LD4 to LD5, Q12 to Q4, R10 to R15, R11 to R16, R12 to R17, R13 to R18, R14 to R19, R15 to R20, R16 to R21, R17 to R22, R18 to R23, R19 to R24, R20 to R25, U6 to U2, U7 to U3, U8 to U4, U9 to U5, U10 to U6, U4 to U7

Commit message: delete unuse
Parts:
- removed C19: 100n, Capacitor_SMD:C_0402_1005Metric, symbol Device:C
- removed JP1: CFG1, Jumper:SolderJumper-2_P1.3mm_Open_RoundedPad1.0x1.5mm, symbol Jumper:SolderJumper_2_Bridged
- removed JP2: CFG2, Jumper:SolderJumper-2_P1.3mm_Open_RoundedPad1.0x1.5mm, symbol Jumper:SolderJumper_2_Open
- removed JP3: CFG3, Jumper:SolderJumper-2_P1.3mm_Open_RoundedPad1.0x1.5mm, symbol Jumper:SolderJumper_2_Open
- removed JP4, JP5, JP6: CFG, Jumper:SolderJumper-2_P1.3mm_Open_RoundedPad1.0x1.5mm, symbol Jumper:SolderJumper_2_Open
- removed LD4: POW_OK, LED_SMD:LED_0603_1608Metric, symbol Device:LED
- removed R16, R17, R18, R19: 10k, Resistor_SMD:R_0603_1608Metric, symbol Device:R
- removed R20: 1k, Resistor_SMD:R_0603_1608Metric, symbol Device:R
- removed R21, R22: 200k, Resistor_SMD:R_0603_1608Metric, symbol Device:R
- removed R24: 68k, Resistor_SMD:R_0603_1608Metric, symbol Device:R
- removed R25: 24k, Resistor_SMD:R_0603_1608Metric, symbol Device:R
- removed U2: CH221K, Package_TO_SOT_SMD:SOT-23-6, symbol Interface_USB:CH221K
- removed U3: CH224K, Package_SO:SSOP-10-1EP_3.9x4.9mm_P1mm_EP2.1x3.3mm, symbol Interface_USB:CH224K
Connections:
- net +5V: no longer C20.1, U6.3 (VI)
- new net VBUS: C20.1, U6.3 (VI)
- no-connect marks 4 -> 2
Other:
- note removed: "CC Controller"
- note removed: "Green"
- note removed: "VBUS Config"
- note removed: "Voltage R JP7 JP8 JP9 5V 10.2k S S S 9V 21.8k O O S 12V 51.7k O S O 15V 100k S O O 20V 200k O O O"

Commit message: update partname
Parts:
- renumbered C20 to C19, C21 to C20, C22 to C21, C23 to C22, JP7 to JP1, LD5 to LD4, R23 to R16, U4 to U2, U5 to U3, U6 to U4, U7 to U5

Commit message: add v0.02
Parts:
- Q4: LCSC (none) -> C20917; akizuki (none) -> x
- U5: value TLV70012_SOT23-5 -> TLV74311PDBVR; LCSC (none) -> C485147; akizuki (none) -> x
Changed lines of the file:
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@@
 	(title_block
 		(title "PicoBPSK")
-		(date "2026-09-03")
-		(rev "0.01")
+		(date "2026-09-07")
+		(rev "0.02")
 		(company "okdwtr")
 		(comment 1 "USB-BPSK Converter Using RP2354")
@@
 			)
 		)
-		(property "Value" "TLV70012_SOT23-5"
+		(property "Value" "TLV74311PDBVR"
 			(at 241.3 133.35 0)
 			(show_name no)
@@
 			)
 		)
+		(property "LCSC" "C485147"
+			(at 241.3 139.7 0)
+			(hide yes)
+			(show_name no)
+			(do_not_autoplace no)
+			(effects
+				(font
+					(size 1.27 1.27)
+				)
+			)
+		)
+		(property "akizuki" "x"
+			(at 241.3 139.7 0)
+			(hide yes)
+			(show_name no)
+			(do_not_autoplace no)
+			(effects
+				(font
+					(size 1.27 1.27)
+				)
+			)
+		)
 		(pin "4"
 		)
@@
 			(at 194.31 139.7 0)
 			(hide yes)
+			(show_name no)
+			(do_not_autoplace no)
+			(effects
+				(font
+					(size 1.27 1.27)
+				)
+			)
+		)
+		(property "LCSC" "C20917"
+			(at 194.31 139.7 0)
+			(hide yes)
+			(show_name no)
+			(do_not_autoplace no)
+			(effects
+				(font
+					(size 1.27 1.27)
+				)
+			)
+		)
+		(property "akizuki" "x"
+			(at 194.31 139.7 0)
+			(hide yes)
